File: psu/iggie_psu.sch (KiCad schematic (older format))
At the start: 58 parts

Commit message: spec most parts
Parts:
- removed C? (x8): 22µ, symbol agg:C
- removed C?: C, symbol agg:C
- removed R?: R, symbol agg:R
- added C11, C8: 10µ, agg:0805, symbol agg:C
- added C20: 100p, symbol agg:C
- added C21, C22: 220n, agg:1206, symbol agg:C
- added C23, C24: 10µ, symbol agg:CP
- added D7, D8: LED, symbol agg:LED
- added IC2: MCP1416, agg:SOT-23-5, symbol agg:MCP1416
- added R1: 100k, agg:0603, symbol agg:R
- added R12, R13: R, symbol agg:R
- added R2: 10k, symbol agg:R
- added R3: 100k, symbol agg:R
- added R9: 2R2, symbol agg:R
- C10, C12, C2, C3, C5, C7: renamed from C?; value C -> 100n; footprint (none) -> agg:0603
- C15, C17: renamed from C?; value C -> 10µ; footprint (none) -> agg:0805; Farnell (none) -> 2611941
- C16: renamed from C?; value C -> 10n; footprint (none) -> agg:0603
- C18: renamed from C?; value C -> 100p; Voltage (none) -> 250V
- C19: renamed from C?; value C -> 100p; footprint (none) -> agg:0603
- C9: renamed from C?; value C -> 4µ7; footprint (none) -> agg:0603
- D6: renamed from D?; footprint (none) -> agg:DO-214AA-SMB; Farnell (none) -> 2675075
- L1: renamed from L?; value L -> 68µ; footprint (none) -> agg:MSS1210; Current (none) -> 3.8A; Farnell (none) -> 2288336
- Q1: renamed from Q?; Farnell (none) -> 2841642
- R10, R7: renamed from R?; value R -> 100m; footprint (none) -> agg:1210
- R11: renamed from R?; value R -> 1k; footprint (none) -> agg:0603
- R14, R15, R16, R17: renamed from R?; value R -> 500k
- R18: renamed from R?; value R -> 10k
- R4: renamed from R?; value R -> 100k; footprint (none) -> agg:0603
- R5: renamed from R?; value R -> 10k; footprint (none) -> agg:0603
- R6: renamed from R?; value 10k -> 100k
- R8: renamed from R?; value R -> 2R2
- Y1: renamed from Y?; value XTAL -> 8M
- gave numbers to parts that had none: 20
Connections:
- net labels added: CP_OUT_MON, OPAMP2_OUT
- net labels removed: CP_OUT, OPAMP2OUT
- wire segments 192 -> 220
- no-connect marks 11 -> 5
Other:
- note added: "18V"
- note added: "400V"
- note added: "= VOUT/201\n= 2V"
- note added: "=CP_OUT/11\n=1.64V"
- note added: "=LI/20\n=0.19V"
- note added: "=VIN/11\n=0.45V"
- note added: "Charge Pump"
- note added: "Divider:\n0.2mA / 80mW"
- note added: "PA0: ADC1_IN1 (FAST)"
- note added: "PA10: TIM2_CH4"
- note added: "PA1: ADC1_IN2 (FAST)"
- note added: "PA3: ADC1_IN4 (FAST)"
- note added: "PA7: ADC2_IN4 (FAST), COMP2_INP, OPAMP2_VINP"
- note added: "PA9: TIM2_CH3"
- note added: "Snubber"
- note removed: "PA0: ADC1_IN1\n"
- note removed: "PA7: ADC2_IN4, COMP2_INP, OPAMP2_VINP"
- moved on the sheet: C1, C15, C17, C18, C19, C2, C3, C4, C5, C6, C7, IC1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

Commit message: add some TPs etc
Parts:
- removed Y1: 8M, symbol agg:XTAL
- added J4: GND, agg:SIL-254P-01, symbol agg:CONN_01x01
- added TP10, TP11, TP12, TP13, TP5, TP6, TP7, TP8, TP9: TESTPAD, agg:TESTPAD, symbol agg:TESTPAD
- added X1, X2, X3, X4: M3 MOUNT, agg:M3_MOUNT, symbol agg:PART
- added Y?: 26M, agg:XTAL-20x16, symbol agg:SMD_XTAL
- C13, C14: value C -> 10p
- C23, C24: Farnell 2326345 -> (none)
- D1, D2, D3, D4, D5, D6: value D -> ~
- D7, D8: footprint (none) -> agg:0603-LED; Farnell (none) -> 2290329
- R12, R13: value R -> 1k; footprint (none) -> agg:0603
- R18, R2, R3, R6: footprint (none) -> agg:0603
Connections:
- wire segments 220 -> 234
Other:
- moved on the sheet: C13, C14, J1
