File: psu_boost/psu.sch (KiCad schematic (older format))
At the start: 57 parts

Commit message: Stop work on 2stage boost, swap to new flyback design
Parts:
- removed C? (x3): 1µ, agg:0603, symbol agg:C
- removed C? (x3): 10µ, agg:1210, symbol agg:C
- removed C? (x4): 100n, agg:0603, symbol agg:C
- removed C?: 100p, agg:0603, symbol agg:C
- removed D? (x3): ESD_DIODE, agg:0603, symbol agg:ESD_DIODE
- removed D?: RED, agg:0603-LED, symbol agg:LED
- removed D? (x7): GRN, agg:0603-LED, symbol agg:LED
- removed D?: VSSC520S-M3/9AT, agg:DO-214AB-SMC, symbol agg:SCHOTTKY
- removed D?: SMAJ58A, agg:DO-214AC-SMA, symbol agg:SCHOTTKY
- removed IC?: STM32F334K8T6, agg:LQFP-32, symbol agg:STM32F3xxKxTx
- removed IC?: TSR 1-2450, agg:TSR1, symbol agg:TSR1
- removed IC?: TSR 1-24150, agg:TSR1, symbol agg:TSR1
- removed IC?: NCP161, agg:SOT-23-5, symbol agg:NCP161
- removed J?: CTRL, agg:MOLEX-KK-254P-04, symbol agg:CONN_01x04
- removed J?: PWR_IN, agg:BARRELJACK, symbol agg:BarrelJack
- removed J?: HV_OUT, agg:MOLEX-KK-254P-03, symbol agg:CONN_01x03
- removed L?: FB, agg:0603, symbol agg:L
- removed P?: SWD, agg:FTSH-105-01-L-DV-K, symbol agg:SWD
- removed R? (x8): 1k, agg:0603, symbol agg:R
- removed R? (x4): 10k, agg:0603, symbol agg:R
- removed R?: 100k, agg:0603, symbol agg:R
- removed TP?: TESTPAD, agg:SIL-254P-01, symbol agg:TESTPAD
- removed TP? (x4): TESTPAD, agg:TESTPAD, symbol agg:TESTPAD
- removed X? (x4): M3 MOUNT, agg:M3_MOUNT, symbol agg:PART
- removed X?: MAINS PSU, symbol agg:PART
- removed Y?: 25M, agg:XTAL-25x20, symbol agg:TCXO_ST
- added C1: 100µ, agg:PANASONIC-SMDCAP-G, symbol agg:CP
- added C10, C12, C13, C9: 100n, agg:0603, symbol agg:C
- added C11, C4, C5: 1µ, agg:0603, symbol agg:C
- added C2, C3, C8: 10µ, agg:1210, symbol agg:C
- added C7: 100p, agg:0603, symbol agg:C
- added D1: VSSC520S-M3/9AT, agg:DO-214AB-SMC, symbol agg:SCHOTTKY
- added D10: RED, agg:0603-LED, symbol agg:LED
- added D11, D12, D13, D3, D4, D5, D6: GRN, agg:0603-LED, symbol agg:LED
- added D2: SMAJ58A, agg:DO-214AC-SMA, symbol agg:SCHOTTKY
- added D7, D8, D9: ESD_DIODE, agg:0603, symbol agg:ESD_DIODE
- added IC1: NCP161, agg:SOT-23-5, symbol agg:NCP161
- added IC2: TSR 1-24150, agg:TSR1, symbol agg:TSR1
- added IC3: TSR 1-2450, agg:TSR1, symbol agg:TSR1
- added IC4: STM32F334K8T6, agg:LQFP-32, symbol agg:STM32F3xxKxTx
- added J1: HV_OUT, agg:MOLEX-KK-254P-03, symbol agg:CONN_01x03
- added J2: PWR_IN, agg:BARRELJACK, symbol agg:BarrelJack
- added J3: CTRL, agg:MOLEX-KK-254P-04, symbol agg:CONN_01x04
- added L3: FB, agg:0603, symbol agg:L
- added P1: SWD, agg:FTSH-105-01-L-DV-K, symbol agg:SWD
- added R1: 100k, agg:0603, symbol agg:R
- added R10, R11, R12, R13, R4, R5, R8, R9: 1k, agg:0603, symbol agg:R
- added R2, R3, R6, R7: 10k, agg:0603, symbol agg:R
- added TP1, TP3, TP4, TP5: TESTPAD, agg:TESTPAD, symbol agg:TESTPAD
- added TP2: TESTPAD, agg:SIL-254P-01, symbol agg:TESTPAD
- added X1, X2, X3, X4: M3 MOUNT, agg:M3_MOUNT, symbol agg:PART
- added X5: MAINS PSU, symbol agg:PART
- added Y1: 25M, agg:XTAL-25x20, symbol agg:TCXO_ST
Connections:
- net 15v: now also IC2.3 (VOUT), R3.1, TP3.1 (TP)
- net 24v: now also C1.2, C2.1, C3.1, D1.1, D9.1, IC2.1 (VIN), IC3.1 (VIN), J3.1, R1.1, R6.1, TP1.1 (TP)
- net 3v3: now also C10.1, C13.1, C5.1, C8.1, C9.1, IC1.5 (OUT), IC4.1 (VDD), IC4.17 (VDD), L3.2, P1.1 (VTref), R5.1, R7.2, TP5.1 (TP), Y1.1 (~ST), Y1.4 (VCC)
- net 5v: now also C4.1, IC1.1 (IN), IC1.3 (EN), IC3.3 (VOUT), R4.1, TP4.1 (TP)
- net GND: now also C1.1, C10.2, C11.2, C12.2, C13.2, C2.2, C3.2, C4.2, C5.2, C7.2, C8.2, C9.2, D10.1, D11.1, D12.1, D13.1, D2.2, D3.1, D4.1, D5.1, D6.1, D7.2, D8.2, D9.2, IC1.2 (GND), IC2.2 (GND), IC3.2 (GND), IC4.16 (VSS), IC4.31 (BOOT0), IC4.32 (VSS), J2.3 (RING), J3.4, P1.3 (GND), P1.5 (GND), P1.9 (GND), R2.2, TP2.1 (TP), Y1.2 (GND)
- net LED_FAULT: now also IC4.30 (PB7), R10.1
- net LED_OK1: now also IC4.27 (PB4), R12.1
- net LED_OK2: now also IC4.28 (PB5), R13.1
- net LED_STAT: now also IC4.26 (PB3), R11.1
- net SWCLK: now also IC4.24 (PA14), P1.4 (SWDCLK/TCK)
- net SWDIO: now also IC4.23 (PA13), P1.2 (SWDIO/TMS)
- net UART_TX: now also IC4.29 (PB6), R9.2
- net ~RST: now also IC4.4 (NRST), P1.10 (nRESET)
- net ~RUN: now also IC4.25 (PA15), R7.1, R8.2
- new net: IC4.2 (PF0), Y1.3 (OUT)
- new net: C11.1, C12.1, IC4.5 (VDDA), L3.1
- new net: D8.1, J3.2, R8.1
- new net: D7.1, J3.3, R9.1
- new net: D1.2, D2.1, J2.1 (TIP)
- new net: D10.2, R10.2
- new net: D11.2, R11.2
- new net: D6.2, R6.2
- new net: D4.2, R4.2
- new net: D5.2, R5.2
- new net: D12.2, R12.2
- new net: D13.2, R13.2
- new net: D3.2, R3.2
- new net 100V_MON: IC4.7 (PA1)
- new net 24VEN: IC4.21 (PA11)
- new net 24V_MON: C7.1, IC4.6 (PA0), R1.2, R2.1
- new net 400V_MON: IC4.8 (PA2)
- new net Boost Converter/HV+: J1.1
- new net Boost Converter/HV-: J1.3
- new net GD1: IC4.18 (PA8)
- new net GD2: IC4.15 (PB1), IC4.20 (PA10)
- new net GD3: IC4.19 (PA9)
- new net I_24V: IC4.9 (PA3)
- new net I_400V: IC4.11 (PA5)
- new net I_L1: IC4.13 (PA7)
- new net I_L2: IC4.12 (PA6), IC4.14 (PB0)
- no-connect marks 12 -> 7
Other:
- note added: "24VDC 2.5A\n2.1mm barrel jack"
- note added: "5V in, 3.3V 0.5A out"
- note added: "High-Voltage Boost Converter"
- note added: "PA10: TIM1_C3/HRTIM1_CB1"
- note added: "PA5: ADC2_C2"
- note added: "PA9: TIM2_C3"
- note added: "PB1: TIM3_C4"
- note removed: "24VDC 2.5A 60W\n2.1mm barrel jack"
- note removed: "5V in, 3.3V 450mA out"
- note removed: "High-Voltage Flyback Converter"
- note removed: "add serial input?\nfewer LEDs?\ninterface to a display?"
