File: driver/iggie-driver.kicad_pcb (KiCad board)
At the start: 2 copper layers, 450 parts, among them IC101 TSR 1-2433, IC102 STM32F405RxTx, IC103 ESP-12, IC1101 74HC595, IC1102 74HC595, IC1103 74HC595, IC1104 74HC595, IC1105 74HC595, IC1106 74HC595, IC1107 74HC595, IC1108 74HC595, IC1109 74HC595, IC1110 74HC595, IC1111 74HC595, IC1112 74HC595, IC1113 74HC595, IC1114 74HC595, IC1115 74HC595, IC1116 74HC595, J101 PSU, J102 HV, J103 DRIVE, J104 DIRECT, J105 UART, J106 ESP_FLASH, J201 A_1_32, J202 A_33_64, J203 K_1_32, J204 K_33_64, P101 SWD, Q1001 PBHV9050T,215, Q1002 PBHV9050T,215, Q1003 PBHV9050T,215, Q1004 PBHV9050T,215, Q1005 DMN60H080DS-7, Q1006 DMN60H080DS-7, Q1007 DMN60H080DS-7, Q1008 DMN60H080DS-7, Q1009 DMN60H080DS-7, Q1010 DMN60H080DS-7, Q1011 DMN60H080DS-7, Q1012 DMN60H080DS-7, Q1013 PBHV9050T,215, Q1014 PBHV9050T,215, Q1015 PBHV9050T,215, Q1016 PBHV9050T,215, Q1017 DMN60H080DS-7, Q1018 DMN60H080DS-7, Q1019 DMN60H080DS-7, Q1020 DMN60H080DS-7, Q1021 DMN60H080DS-7, Q1022 DMN60H080DS-7, Q1023 DMN60H080DS-7, Q1024 DMN60H080DS-7, Q301 PBHV9050T,215, Q302 PBHV9050T,215, Q303 PBHV9050T,215, Q304 PBHV9050T,215, Q305 DMN60H080DS-7, Q306 DMN60H080DS-7, Q307 DMN60H080DS-7, Q308 DMN60H080DS-7, Q309 DMN60H080DS-7, Q310 DMN60H080DS-7, Q311 DMN60H080DS-7, Q312 DMN60H080DS-7, Q313 PBHV9050T,215, Q314 PBHV9050T,215, Q315 PBHV9050T,215, Q316 PBHV9050T,215, Q317 DMN60H080DS-7, Q318 DMN60H080DS-7, Q319 DMN60H080DS-7, Q320 DMN60H080DS-7, Q321 DMN60H080DS-7, Q322 DMN60H080DS-7, Q323 DMN60H080DS-7, Q324 DMN60H080DS-7, Q401 PBHV9050T,215, Q402 PBHV9050T,215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

Commit message: WIP PCB
Parts:
- added X101: M3 MOUNT, agg:M3_MOUNT, F.Cu at (52.0, 52.0)
- added X102: M3 MOUNT, agg:M3_MOUNT, F.Cu at (200.0, 52.0)
- added X103: M3 MOUNT, agg:M3_MOUNT, F.Cu at (200.0, 200.0)
- added X104: M3 MOUNT, agg:M3_MOUNT, F.Cu at (52.0, 200.0)
- added X105: M3 MOUNT, agg:M3_MOUNT, F.Cu at (80.0, 80.0)
- added X106: M3 MOUNT, agg:M3_MOUNT, F.Cu at (172.0, 80.0)
- added X107: M3 MOUNT, agg:M3_MOUNT, F.Cu at (172.0, 172.0)
- added X108: M3 MOUNT, agg:M3_MOUNT, F.Cu at (80.0, 172.0)
- Q306, Q308, Q314, Q316, Q318, Q320, R304, R306, R308, R314, R316, R318, R320: moved to B.Cu
- moved IC103 225.7 mm to (259.7, 163.8), turned to 180 degrees
- moved J106 194.4 mm to (262.3, 141.6)
- moved R522 164.5 mm to (86.5, 156.0), turned to 180 degrees
- moved R511 162.5 mm to (86.5, 158.5), turned to 180 degrees
- moved R509 157.6 mm to (86.5, 163.5), turned to 180 degrees
- moved C108 154.4 mm to (95.8, -95.9)
- moved C1107 154.4 mm to (141.9, -98.4)
- moved C1114 154.4 mm to (146.0, -98.4)
- moved C112 154.4 mm to (91.7, -95.9)
- moved C114 154.4 mm to (87.6, -95.9)
- moved Q1007 154.4 mm to (170.4, -9.58)
- moved Q1008 154.4 mm to (181.8, -20.7)
- moved Q1011 154.4 mm to (171.3, -14.1)
- moved Q1012 154.4 mm to (160.8, -13.2)
- moved Q1015 154.4 mm to (177.0, -20.7)
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Connections:
- C101 pad 2: 24v -> GND
- C102 pad 2: 24v -> GND
- C103 pad 2: 24v -> GND
- C104 pad 2: 24v -> GND
- C105 pad 2: 24v -> GND
- C106 pad 2: 24v -> GND
- C107 pad 2: 24v -> GND
- C108 pad 2: 24v -> GND
- C109 pad 2: 24v -> GND
- C110 pad 2: 24v -> GND
- C1101 pad 2: 24v -> GND
- C1102 pad 2: 24v -> GND
- C1103 pad 2: 24v -> GND
- C1104 pad 2: 24v -> GND
- C1105 pad 2: 24v -> GND
- C1106 pad 2: 24v -> GND
- C1107 pad 2: 24v -> GND
- C1108 pad 2: 24v -> GND
- C1109 pad 2: 24v -> GND
- C111 pad 2: 24v -> GND
- C1110 pad 2: 24v -> GND
- C1111 pad 2: 24v -> GND
- C1112 pad 2: 24v -> GND
- C1113 pad 2: 24v -> GND
- C1114 pad 2: 24v -> GND
- C1115 pad 2: 24v -> GND
- C1116 pad 2: 24v -> GND
- C112 pad 2: 24v -> GND
- C113 pad 2: 24v -> GND
- C114 pad 2: 24v -> GND
- D101 pad 2: 24v -> GND
- D102 pad 2: 24v -> GND
- D103 pad 2: 24v -> GND
- IC101 pad 2: 24v -> GND
- IC102 pad 12: 24v -> GND
- IC102 pad 18: 24v -> GND
- IC102 pad 60: 24v -> GND
- IC102 pad 63: 24v -> GND
- IC103 pad 15: 24v -> GND
- IC1101 pad 8: 24v -> GND
- IC1102 pad 8: 24v -> GND
- IC1103 pad 8: 24v -> GND
- IC1104 pad 8: 24v -> GND
- IC1105 pad 8: 24v -> GND
- IC1106 pad 8: 24v -> GND
- IC1107 pad 8: 24v -> GND
- IC1108 pad 8: 24v -> GND
- IC1109 pad 8: 24v -> GND
- IC1110 pad 8: 24v -> GND
- IC1111 pad 8: 24v -> GND
- IC1112 pad 8: 24v -> GND
- IC1113 pad 8: 24v -> GND
- IC1114 pad 8: 24v -> GND
- IC1115 pad 8: 24v -> GND
- IC1116 pad 8: 24v -> GND
- J101 pad 4: 24v -> GND
- J102 pad 1: 400V -> GND
- J102 pad 3: 24v -> 400V
- J103 pad 15: 24v -> GND
- J103 pad 16: 24v -> GND
- J104 pad 8: 24v -> GND
- J105 pad 4: 24v -> GND
- J106 pad 2: Net-(IC103-Pad10) -> Net-(IC103-Pad13)
- J106 pad 3: Net-(IC103-Pad13) -> Net-(IC103-Pad10)
- J106 pad 5: 24v -> GND
- J203 pad 1: /Channels/K1 -> /Channels/K31
- J203 pad 10: /Channels/K10 -> /Channels/K22
- J203 pad 11: /Channels/K11 -> /Channels/K21
- J203 pad 12: /Channels/K12 -> /Channels/K26
- J203 pad 13: /Channels/K13 -> /Channels/K19
- J203 pad 14: /Channels/K14 -> /Channels/K20
- J203 pad 15: /Channels/K15 -> /Channels/K17
- J203 pad 16: /Channels/K16 -> /Channels/K18
- J203 pad 17: /Channels/K17 -> /Channels/K15
- J203 pad 18: /Channels/K18 -> /Channels/K16
- J203 pad 19: /Channels/K19 -> /Channels/K13
- J203 pad 2: /Channels/K2 -> /Channels/K32
- J203 pad 20: /Channels/K20 -> /Channels/K14
- J203 pad 21: /Channels/K21 -> /Channels/K11
- J203 pad 22: /Channels/K26 -> /Channels/K12
- J203 pad 23: /Channels/K23 -> /Channels/K9
- J203 pad 24: /Channels/K22 -> /Channels/K10
- J203 pad 25: /Channels/K25 -> /Channels/K7
- J203 pad 26: /Channels/K28 -> /Channels/K8
- J203 pad 27: /Channels/K27 -> /Channels/K5
- J203 pad 28: /Channels/K24 -> /Channels/K6
- J203 pad 29: /Channels/K29 -> /Channels/K3
- J203 pad 3: /Channels/K3 -> /Channels/K29
- J203 pad 30: /Channels/K30 -> /Channels/K4
- J203 pad 31: /Channels/K31 -> /Channels/K1
- J203 pad 32: /Channels/K32 -> /Channels/K2
- J203 pad 4: /Channels/K4 -> /Channels/K30
- J203 pad 5: /Channels/K5 -> /Channels/K27
- J203 pad 6: /Channels/K6 -> /Channels/K24
- J203 pad 7: /Channels/K7 -> /Channels/K25
- J203 pad 8: /Channels/K8 -> /Channels/K28
- J203 pad 9: /Channels/K9 -> /Channels/K23
- J204 pad 1: /Channels/K33 -> /Channels/K63
- J204 pad 10: /Channels/K42 -> /Channels/K56
- J204 pad 11: /Channels/K43 -> /Channels/K53
- J204 pad 12: /Channels/K44 -> /Channels/K54
- J204 pad 13: /Channels/K45 -> /Channels/K51
- J204 pad 14: /Channels/K46 -> /Channels/K52
- J204 pad 15: /Channels/K47 -> /Channels/K49
- J204 pad 16: /Channels/K48 -> /Channels/K50
- J204 pad 17: /Channels/K49 -> /Channels/K47
- J204 pad 18: /Channels/K50 -> /Channels/K48
- J204 pad 19: /Channels/K51 -> /Channels/K45
- J204 pad 2: /Channels/K34 -> /Channels/K64
- J204 pad 20: /Channels/K52 -> /Channels/K46
- J204 pad 21: /Channels/K53 -> /Channels/K43
- J204 pad 22: /Channels/K54 -> /Channels/K44
- J204 pad 23: /Channels/K55 -> /Channels/K41
- J204 pad 24: /Channels/K56 -> /Channels/K42
- J204 pad 25: /Channels/K57 -> /Channels/K39
- J204 pad 26: /Channels/K58 -> /Channels/K40
- J204 pad 27: /Channels/K59 -> /Channels/K37
- J204 pad 28: /Channels/K60 -> /Channels/K38
- J204 pad 29: /Channels/K61 -> /Channels/K35
- J204 pad 3: /Channels/K35 -> /Channels/K61
- J204 pad 30: /Channels/K62 -> /Channels/K36
- J204 pad 31: /Channels/K63 -> /Channels/K33
- J204 pad 32: /Channels/K64 -> /Channels/K34
- J204 pad 4: /Channels/K36 -> /Channels/K62
- J204 pad 5: /Channels/K37 -> /Channels/K59
- J204 pad 6: /Channels/K38 -> /Channels/K60
- J204 pad 7: /Channels/K39 -> /Channels/K57
- J204 pad 8: /Channels/K40 -> /Channels/K58
- J204 pad 9: /Channels/K41 -> /Channels/K55
- P101 pad 3: 24v -> GND
- P101 pad 5: 24v -> GND
- P101 pad 9: 24v -> GND
- Q1005 pad 2: 24v -> GND
- Q1006 pad 2: 24v -> GND
- Q1007 pad 2: 24v -> GND
- Q1008 pad 2: 24v -> GND
- Q1009 pad 2: 24v -> GND
- Q1010 pad 2: 24v -> GND
- Q1011 pad 2: 24v -> GND
- Q1012 pad 2: 24v -> GND
- Q1017 pad 2: 24v -> GND
- Q1018 pad 2: 24v -> GND
- Q1019 pad 2: 24v -> GND
- Q1020 pad 2: 24v -> GND
- Q1021 pad 2: 24v -> GND
- Q1022 pad 2: 24v -> GND
- Q1023 pad 2: 24v -> GND
- Q1024 pad 2: 24v -> GND
- Q305 pad 2: 24v -> GND
- Q306 pad 2: 24v -> GND
- Q307 pad 2: 24v -> GND
- Q308 pad 2: 24v -> GND
- Q309 pad 2: 24v -> GND
- Q310 pad 2: 24v -> GND
- Q311 pad 2: 24v -> GND
- Q312 pad 2: 24v -> GND
- Q317 pad 2: 24v -> GND
- Q318 pad 2: 24v -> GND
- Q319 pad 2: 24v -> GND
- Q320 pad 2: 24v -> GND
- Q321 pad 2: 24v -> GND
- Q322 pad 2: 24v -> GND
- Q323 pad 2: 24v -> GND
- Q324 pad 2: 24v -> GND
- Q405 pad 2: 24v -> GND
- Q406 pad 2: 24v -> GND
- Q407 pad 2: 24v -> GND
- Q408 pad 2: 24v -> GND
- Q409 pad 2: 24v -> GND
- Q410 pad 2: 24v -> GND
- Q411 pad 2: 24v -> GND
- Q412 pad 2: 24v -> GND
- Q417 pad 2: 24v -> GND
- Q418 pad 2: 24v -> GND
- Q419 pad 2: 24v -> GND
- Q420 pad 2: 24v -> GND
- Q421 pad 2: 24v -> GND
- Q422 pad 2: 24v -> GND
- Q423 pad 2: 24v -> GND
- Q424 pad 2: 24v -> GND
- Q505 pad 2: 24v -> GND
- Q506 pad 2: 24v -> GND
- Q507 pad 2: 24v -> GND
- Q508 pad 2: 24v -> GND
- Q509 pad 2: 24v -> GND
- Q510 pad 2: 24v -> GND
- Q511 pad 2: 24v -> GND
- Q512 pad 2: 24v -> GND
- Q517 pad 2: 24v -> GND
- Q518 pad 2: 24v -> GND
- Q519 pad 2: 24v -> GND
- Q520 pad 2: 24v -> GND
- Q521 pad 2: 24v -> GND
- Q522 pad 2: 24v -> GND
- Q523 pad 2: 24v -> GND
- Q524 pad 2: 24v -> GND
- Q605 pad 2: 24v -> GND
- Q606 pad 2: 24v -> GND
- Q607 pad 2: 24v -> GND
- Q608 pad 2: 24v -> GND
- Q609 pad 2: 24v -> GND
- Q610 pad 2: 24v -> GND
- Q611 pad 2: 24v -> GND
- Q612 pad 2: 24v -> GND
- Q617 pad 2: 24v -> GND
- Q618 pad 2: 24v -> GND
- Q619 pad 2: 24v -> GND
- Q620 pad 2: 24v -> GND
- Q621 pad 2: 24v -> GND
- Q622 pad 2: 24v -> GND
- Q623 pad 2: 24v -> GND
- Q624 pad 2: 24v -> GND
- Q705 pad 2: 24v -> GND
- Q706 pad 2: 24v -> GND
- Q707 pad 2: 24v -> GND
- Q708 pad 2: 24v -> GND
- Q709 pad 2: 24v -> GND
- Q710 pad 2: 24v -> GND
- Q711 pad 2: 24v -> GND
- Q712 pad 2: 24v -> GND
- Q717 pad 2: 24v -> GND
- Q718 pad 2: 24v -> GND
- Q719 pad 2: 24v -> GND
- Q720 pad 2: 24v -> GND
- Q721 pad 2: 24v -> GND
- Q722 pad 2: 24v -> GND
- Q723 pad 2: 24v -> GND
- Q724 pad 2: 24v -> GND
- Q805 pad 2: 24v -> GND
- Q806 pad 2: 24v -> GND
- Q807 pad 2: 24v -> GND
- Q808 pad 2: 24v -> GND
- Q809 pad 2: 24v -> GND
- Q810 pad 2: 24v -> GND
- Q811 pad 2: 24v -> GND
- Q812 pad 2: 24v -> GND
- Q817 pad 2: 24v -> GND
- Q818 pad 2: 24v -> GND
- Q819 pad 2: 24v -> GND
- Q820 pad 2: 24v -> GND
- Q821 pad 2: 24v -> GND
- Q822 pad 2: 24v -> GND
- Q823 pad 2: 24v -> GND
- Q824 pad 2: 24v -> GND
- Q905 pad 2: 24v -> GND
- Q906 pad 2: 24v -> GND
- Q907 pad 2: 24v -> GND
- Q908 pad 2: 24v -> GND
- Q909 pad 2: 24v -> GND
- Q910 pad 2: 24v -> GND
- Q911 pad 2: 24v -> GND
- Q912 pad 2: 24v -> GND
- Q917 pad 2: 24v -> GND
- Q918 pad 2: 24v -> GND
- Q919 pad 2: 24v -> GND
- Q920 pad 2: 24v -> GND
- Q921 pad 2: 24v -> GND
- Q922 pad 2: 24v -> GND
- Q923 pad 2: 24v -> GND
- Q924 pad 2: 24v -> GND
- Y101 pad 2: 24v -> GND
Other:
- board outline added: 162.1 x 162.1 mm
- rule via_min_size: 0.4 -> 0.6
- board text added: "A1"
- board text added: "A64"
- board text added: "K1"
- board text added: "K64"

Commit message: Start work on 32ch board
Parts:
- removed C1101, C1102, C1103, C1104, C1105, C1106, C1107, C1108, C1109, C1110, C1111, C1112, C1113, C1114, C1115, C1116: 100n, agg:0603
- removed IC1101, IC1102, IC1103, IC1104, IC1105, IC1106, IC1107, IC1108, IC1109, IC1110, IC1111, IC1112, IC1113, IC1114, IC1115, IC1116: 74HC595, agg:TSSOP-16
- removed J203: K_1_32, agg:DIL-254P-32
- removed J204: K_33_64, agg:DIL-254P-32
- removed Q1001, Q1002, Q1003, Q1004, Q1013, Q1014, Q1015, Q1016, Q701, Q702, Q703, Q704, Q713, Q714, Q715, Q716, Q801, Q802, Q803, Q804, Q813, Q814, Q815, Q816, Q901, Q902, Q903, Q904, Q913, Q914, Q915, Q916: PBHV9050T,215, agg:SOT-23
- removed Q1005, Q1006, Q1007, Q1008, Q1009, Q1010, Q1011, Q1012, Q1017, Q1018, Q1019, Q1020, Q1021, Q1022, Q1023, Q1024, Q705, Q706, Q707, Q708, Q709, Q710, Q711, Q712, Q717, Q718, Q719, Q720, Q721, Q722, Q723, Q724, Q805, Q806, Q807, Q808, Q809, Q810, Q811, Q812, Q817, Q818, Q819, Q820, Q821, Q822, Q823, Q824, Q905, Q906, Q907, Q908, Q909, Q910, Q911, Q912, Q917, Q918, Q919, Q920, Q921, Q922, Q923, Q924: DMN60H080DS-7, agg:SOT-23
- removed R1001, R1002, R1003, R1004, R1005, R1006, R1007, R1008, R1013, R1014, R1015, R1016, R1017, R1018, R1019, R1020, R701, R702, R703, R704, R705, R706, R707, R708, R713, R714, R715, R716, R717, R718, R719, R720, R801, R802, R803, R804, R805, R806, R807, R808, R813, R814, R815, R816, R817, R818, R819, R820, R901, R902, R903, R904, R905, R906, R907, R908, R913, R914, R915, R916, R917, R918, R919, R920: 10k, agg:1206
- removed R1009, R1010, R1011, R1012, R1021, R1022, R1023, R1024, R709, R710, R711, R712, R721, R722, R723, R724, R809, R810, R811, R812, R821, R822, R823, R824, R909, R910, R911, R912, R921, R922, R923, R924: 93k1, agg:1206
- added C115: 100n, agg:0603, F.Cu at (106.1, -35.4)
- added C701: 100n, agg:0603, F.Cu at (204.2, -56.4)
- added C702: 100n, agg:0603, F.Cu at (204.2, -61.4)
- added C703: 100n, agg:0603, F.Cu at (208.3, -58.9)
- added C704: 100n, agg:0603, F.Cu at (199.7, -48.2)
- added C705: 100n, agg:0603, F.Cu at (195.6, -45.7)
- added C706: 100n, agg:0603, F.Cu at (204.2, -58.9)
- added C707: 100n, agg:0603, F.Cu at (195.6, -48.2)
- added C708: 100n, agg:0603, F.Cu at (208.3, -61.4)
- added IC104: ESP-12, agg:ESP-12, F.Cu at (62.5, -53.2)
- added IC701: 74HC595, agg:TSSOP-16, F.Cu at (189.3, -59.4)
- added IC702: 74HC595, agg:TSSOP-16, F.Cu at (180.7, -52.8)
- added IC703: 74HC595, agg:TSSOP-16, F.Cu at (180.7, -59.4)
- added IC704: 74HC595, agg:TSSOP-16, F.Cu at (180.7, -46.2)
- added IC705: 74HC595, agg:TSSOP-16, F.Cu at (189.3, -52.8)
- added IC706: 74HC595, agg:TSSOP-16, F.Cu at (197.9, -59.4)
- added IC707: 74HC595, agg:TSSOP-16, F.Cu at (189.3, -46.2)
- added IC708: 74HC595, agg:TSSOP-16, F.Cu at (197.9, -52.8)
- added J107: ESP_FLASH, agg:SIL-254P-05, F.Cu at (81.3, -39.8)
- C101: value 10µ -> 100n; footprint agg:1210 -> agg:0603
- C102: value 10µ -> 2µ2; footprint agg:1210 -> agg:0603
- C105, C107, C112: value 100n -> 2µ2
- C108, C113: value 2µ2 -> 100n
- C110, C111: value 2µ2 -> 10µ; footprint agg:0603 -> agg:1210
- IC101: value TSR 1-2433 -> STM32F405RxTx; footprint agg:TSR1 -> agg:LQFP-64
- IC102: value STM32F405RxTx -> TSR 1-2433; footprint agg:LQFP-64 -> agg:TSR1
- IC103: value ESP-12 -> ADuM1201; footprint agg:ESP-12 -> agg:SOIC-8
- J103: value DRIVE -> SREG_IN; footprint agg:DIL-254P-16 -> agg:MOLEX-PICOBLADE-53398-0871
- J104: value DIRECT -> DRIVE; footprint agg:MOLEX-PICOBLADE-53398-0871 -> agg:DIL-254P-16
- J106: value ESP_FLASH -> SREG_OUT; footprint agg:SIL-254P-05 -> agg:MOLEX-PICOBLADE-53398-0871
- J202: value A_33_64 -> K_1_32
- Q301, Q302, Q304, Q313, Q401, Q402, Q404, Q413, Q414, Q416, Q501, Q502, Q504, Q513, Q514, Q516, Q601, Q602, Q604, Q613, Q614, Q616: value PBHV9050T,215 -> DMN60H080DS-7
- Q305, Q309, Q311, Q317, Q321, Q323, Q405, Q409, Q411, Q417, Q421, Q423, Q505, Q509, Q511, Q517, Q521, Q523, Q605, Q609, Q611, Q617, Q621, Q623: value DMN60H080DS-7 -> PBHV9050T,215
- Q306, Q308, Q318, Q320, R304, R308, R314, R316, R320: moved to F.Cu
- Q314, Q316: value PBHV9050T,215 -> DMN60H080DS-7; moved to F.Cu
- R305, R317, R405, R406, R417, R418, R505, R506, R517, R518, R605, R606, R617, R618: value 10k -> 93k1
- R306, R318: value 10k -> 93k1; moved to F.Cu
- R309, R310, R321, R322, R409, R410, R421, R422, R509, R510, R521, R522, R609, R610, R621, R622: value 93k1 -> 10k
- moved IC102 286.4 mm to (183.5, 160.0), turned to 270 degrees
- moved R505 271.9 mm to (93.0, 140.0), turned to 180 degrees
- moved Q316 270.8 mm to (168.1, -55.9), turned to 0 degrees
- moved IC103 265.2 mm to (74.0, -25.6), turned to 0 degrees
- moved J106 262.9 mm to (61.0, -27.4)
- moved Q306 261.6 mm to (147.1, -46.0), turned to 0 degrees
- moved Q318 257.3 mm to (161.5, -46.9), turned to 0 degrees
- moved R401 252.2 mm to (108.5, 172.0), turned to 180 degrees
- moved R517 251.9 mm to (93.0, 132.0), turned to 180 degrees
- moved R506 251.8 mm to (93.0, 124.0), turned to 180 degrees
- moved Q403 251.6 mm to (97.5, 172.5), turned to 180 degrees
- moved Q409 250.6 mm to (97.5, 168.5), turned to 180 degrees
- moved R518 250.4 mm to (93.0, 116.0), turned to 180 degrees
- moved Q407 249.8 mm to (113.0, 168.5), turned to 180 degrees
- moved R403 249.6 mm to (103.5, 172.0), turned to 180 degrees
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Connections:
- C101 pad 1: 24v -> 3v3
- C107 pad 1: 3v3 -> Net-(C107-Pad1)
- C109 pad 1: 3v3 -> Net-(C109-Pad1)
- C110 pad 1: Net-(C110-Pad1) -> 24v
- C111 pad 1: Net-(C111-Pad1) -> 3v3
- C112 pad 1: 3v3 -> Net-(C112-Pad1)
- C113 pad 1: Net-(C113-Pad1) -> 3v3
- C114 pad 1: Net-(C113-Pad1) -> Net-(C112-Pad1)
- IC101 pad 1: 24v -> 3v3
- IC101 pad 2: GND -> Net-(IC101-Pad2)
- IC101 pad 3: 3v3 -> Net-(IC101-Pad3)
- IC102 pad 1: 3v3 -> 24v
- IC102 pad 2: Net-(IC102-Pad2) -> GND
- IC102 pad 3: Net-(IC102-Pad3) -> 3v3
- IC103 pad 1: /ESP_~RST -> 3v3
- IC103 pad 2: Net-(IC103-Pad2) -> /UART_RX
- IC103 pad 3: /ESP_EN -> /UART_TX
- IC103 pad 4: Net-(IC103-Pad4) -> GND
- IC103 pad 5: Net-(IC103-Pad5) -> Net-(C115-Pad2)
- IC103 pad 8: Net-(C113-Pad1) -> Net-(C115-Pad1)
- J103 pad 1: /STM32_ACLK -> /ACLK
- J103 pad 2: /ACLK -> /ADAT
- J103 pad 3: /STM32_ADAT -> /KCLK
- J103 pad 4: /ADAT -> /KDAT
- J103 pad 5: /STM32_KCLK -> /STCP
- J103 pad 6: /KCLK -> /~OE
- J103 pad 7: /STM32_KDAT -> /~MR
- J103 pad 8: /KDAT -> GND
- J104 pad 1: /ACLK -> /STM32_ACLK
- J104 pad 2: /ADAT -> /ACLK
- J104 pad 3: /KCLK -> /STM32_ADAT
- J104 pad 4: /KDAT -> /ADAT
- J104 pad 5: /STCP -> /STM32_KCLK
- J104 pad 6: /~OE -> /KCLK
- J104 pad 7: /~MR -> /STM32_KDAT
- J104 pad 8: GND -> /KDAT
- J105 pad 1: 3v3 -> Net-(C115-Pad1)
- J105 pad 2: /UART_RX -> Net-(IC103-Pad7)
- J105 pad 3: /UART_TX -> Net-(IC103-Pad6)
- J105 pad 4: GND -> Net-(C115-Pad2)
- J106 pad 1: Net-(IC103-Pad14) -> /ACLK
- J106 pad 2: Net-(IC103-Pad13) -> /Channels/AOUT
- J106 pad 3: Net-(IC103-Pad10) -> /KCLK
- J106 pad 4: Net-(IC103-Pad9) -> /Channels/KOUT
- J106 pad 5: GND -> /STCP
- J202 pad 1: /Channels/A33 -> /Channels/K31
- J202 pad 10: /Channels/A42 -> /Channels/K22
- J202 pad 11: /Channels/A43 -> /Channels/K21
- J202 pad 12: /Channels/A44 -> /Channels/K26
- J202 pad 13: /Channels/A45 -> /Channels/K19
- J202 pad 14: /Channels/A46 -> /Channels/K20
- J202 pad 15: /Channels/A47 -> /Channels/K17
- J202 pad 16: /Channels/A48 -> /Channels/K18
- J202 pad 17: /Channels/A49 -> /Channels/K15
- J202 pad 18: /Channels/A50 -> /Channels/K16
- J202 pad 19: /Channels/A51 -> /Channels/K13
- J202 pad 2: /Channels/A34 -> /Channels/K32
- J202 pad 20: /Channels/A52 -> /Channels/K14
- J202 pad 21: /Channels/A53 -> /Channels/K11
- J202 pad 22: /Channels/A54 -> /Channels/K12
- J202 pad 23: /Channels/A55 -> /Channels/K9
- J202 pad 24: /Channels/A56 -> /Channels/K10
- J202 pad 25: /Channels/A57 -> /Channels/K7
- J202 pad 26: /Channels/A58 -> /Channels/K8
- J202 pad 27: /Channels/A59 -> /Channels/K5
- J202 pad 28: /Channels/A60 -> /Channels/K6
- J202 pad 29: /Channels/A61 -> /Channels/K3
- J202 pad 3: /Channels/A35 -> /Channels/K29
- J202 pad 30: /Channels/A62 -> /Channels/K4
- J202 pad 31: /Channels/A63 -> /Channels/K1
- J202 pad 32: /Channels/A64 -> /Channels/K2
- J202 pad 4: /Channels/A36 -> /Channels/K30
- J202 pad 5: /Channels/A37 -> /Channels/K27
- J202 pad 6: /Channels/A38 -> /Channels/K24
- J202 pad 7: /Channels/A39 -> /Channels/K25
- J202 pad 8: /Channels/A40 -> /Channels/K28
- J202 pad 9: /Channels/A41 -> /Channels/K23
- L101 pad 2: Net-(C113-Pad1) -> Net-(C112-Pad1)
- Q301 pad 1: Net-(Q301-Pad1) -> /Channels/GA1
- Q301 pad 2: 400V -> GND
- Q302 pad 1: Net-(Q302-Pad1) -> /Channels/GA5
- Q302 pad 2: 400V -> GND
- Q304 pad 1: Net-(Q304-Pad1) -> /Channels/GK1
- Q304 pad 2: 400V -> GND
- Q304 pad 3: Net-(Q304-Pad3) -> /Channels/K1
- Q305 pad 1: /Channels/GA1 -> Net-(Q305-Pad1)
- Q305 pad 2: GND -> 400V
- Q306 pad 1: /Channels/GA2 -> /Channels/GK5
- Q306 pad 3: Net-(Q306-Pad3) -> /Channels/K5
- Q307 pad 1: /Channels/GA3 -> /Channels/GA2
- Q308 pad 1: /Channels/GA4 -> /Channels/GA6
- Q309 pad 1: /Channels/GK1 -> Net-(Q309-Pad1)
- Q309 pad 2: GND -> 400V
- Q309 pad 3: /Channels/K1 -> Net-(Q309-Pad3)
- Q311 pad 1: /Channels/GK3 -> Net-(Q311-Pad1)
- Q311 pad 2: GND -> 400V
- Q311 pad 3: /Channels/K3 -> Net-(Q311-Pad3)
- Q312 pad 1: /Channels/GK4 -> /Channels/GK6
- Q312 pad 3: /Channels/K4 -> /Channels/K6
- Q313 pad 1: Net-(Q313-Pad1) -> /Channels/GA3
- Q313 pad 2: 400V -> GND
- Q314 pad 1: Net-(Q314-Pad1) -> /Channels/GA7
- Q314 pad 2: 400V -> GND
- Q316 pad 1: Net-(Q316-Pad1) -> /Channels/GK3
- Q316 pad 2: 400V -> GND
- Q316 pad 3: Net-(Q316-Pad3) -> /Channels/K3
- Q317 pad 1: /Channels/GA5 -> Net-(Q317-Pad1)
- Q317 pad 2: GND -> 400V
- Q318 pad 1: /Channels/GA6 -> /Channels/GK7
- Q318 pad 3: Net-(Q318-Pad3) -> /Channels/K7
- Q319 pad 1: /Channels/GA7 -> /Channels/GA4
- Q321 pad 1: /Channels/GK5 -> Net-(Q321-Pad1)
- Q321 pad 2: GND -> 400V
- Q321 pad 3: /Channels/K5 -> Net-(Q321-Pad3)
- Q322 pad 1: /Channels/GK6 -> /Channels/GK4
- Q322 pad 3: /Channels/K6 -> /Channels/K4
- Q323 pad 1: /Channels/GK7 -> Net-(Q323-Pad1)
- Q323 pad 2: GND -> 400V
- Q323 pad 3: /Channels/K7 -> Net-(Q323-Pad3)
- Q401 pad 1: Net-(Q401-Pad1) -> /Channels/GA9
- Q401 pad 2: 400V -> GND
- Q402 pad 1: Net-(Q402-Pad1) -> /Channels/GA13
- Q402 pad 2: 400V -> GND
- Q404 pad 1: Net-(Q404-Pad1) -> /Channels/GK9
- Q404 pad 2: 400V -> GND
- Q404 pad 3: Net-(Q404-Pad3) -> /Channels/K9
- Q405 pad 1: /Channels/GA9 -> Net-(Q405-Pad1)
- Q405 pad 2: GND -> 400V
- Q406 pad 1: /Channels/GA10 -> /Channels/GK13
- Q406 pad 3: Net-(Q406-Pad3) -> /Channels/K13
- Q407 pad 1: /Channels/GA11 -> /Channels/GA10
- Q408 pad 1: /Channels/GA12 -> /Channels/GA14
- Q409 pad 1: /Channels/GK9 -> Net-(Q409-Pad1)
- Q409 pad 2: GND -> 400V
- Q409 pad 3: /Channels/K9 -> Net-(Q409-Pad3)
- Q411 pad 1: /Channels/GK11 -> Net-(Q411-Pad1)
- Q411 pad 2: GND -> 400V
- Q411 pad 3: /Channels/K11 -> Net-(Q411-Pad3)
- Q412 pad 1: /Channels/GK12 -> /Channels/GK14
- Q412 pad 3: /Channels/K12 -> /Channels/K14
- Q413 pad 1: Net-(Q413-Pad1) -> /Channels/GA11
- Q413 pad 2: 400V -> GND
- Q414 pad 1: Net-(Q414-Pad1) -> /Channels/GA15
- Q414 pad 2: 400V -> GND
- Q416 pad 1: Net-(Q416-Pad1) -> /Channels/GK11
- Q416 pad 2: 400V -> GND
- Q416 pad 3: Net-(Q416-Pad3) -> /Channels/K11
- Q417 pad 1: /Channels/GA13 -> Net-(Q417-Pad1)
- Q417 pad 2: GND -> 400V
- Q418 pad 1: /Channels/GA14 -> /Channels/GK15
- Q418 pad 3: Net-(Q418-Pad3) -> /Channels/K15
- Q419 pad 1: /Channels/GA15 -> /Channels/GA12
- Q421 pad 1: /Channels/GK13 -> Net-(Q421-Pad1)
- Q421 pad 2: GND -> 400V
- Q421 pad 3: /Channels/K13 -> Net-(Q421-Pad3)
- Q422 pad 1: /Channels/GK14 -> /Channels/GK12
- Q422 pad 3: /Channels/K14 -> /Channels/K12
- Q423 pad 1: /Channels/GK15 -> Net-(Q423-Pad1)
- Q423 pad 2: GND -> 400V
- Q423 pad 3: /Channels/K15 -> Net-(Q423-Pad3)
- Q501 pad 1: Net-(Q501-Pad1) -> /Channels/GA17
- Q501 pad 2: 400V -> GND
- Q502 pad 1: Net-(Q502-Pad1) -> /Channels/GA21
- Q502 pad 2: 400V -> GND
- Q504 pad 1: Net-(Q504-Pad1) -> /Channels/GK17
- Q504 pad 2: 400V -> GND
- Q504 pad 3: Net-(Q504-Pad3) -> /Channels/K17
- Q505 pad 1: /Channels/GA17 -> Net-(Q505-Pad1)
- Q505 pad 2: GND -> 400V
- Q506 pad 1: /Channels/GA18 -> /Channels/GK21
- Q506 pad 3: Net-(Q506-Pad3) -> /Channels/K21
- Q507 pad 1: /Channels/GA19 -> /Channels/GA18
- Q508 pad 1: /Channels/GA20 -> /Channels/GA22
- Q509 pad 1: /Channels/GK17 -> Net-(Q509-Pad1)
- Q509 pad 2: GND -> 400V
- Q509 pad 3: /Channels/K17 -> Net-(Q509-Pad3)
- Q511 pad 1: /Channels/GK19 -> Net-(Q511-Pad1)
- Q511 pad 2: GND -> 400V
- Q511 pad 3: /Channels/K19 -> Net-(Q511-Pad3)
- Q512 pad 1: /Channels/GK20 -> /Channels/GK22
- Q512 pad 3: /Channels/K20 -> /Channels/K22
- Q513 pad 1: Net-(Q513-Pad1) -> /Channels/GA19
- Q513 pad 2: 400V -> GND
- Q514 pad 1: Net-(Q514-Pad1) -> /Channels/GA23
- Q514 pad 2: 400V -> GND
- Q516 pad 1: Net-(Q516-Pad1) -> /Channels/GK19
- Q516 pad 2: 400V -> GND
- Q516 pad 3: Net-(Q516-Pad3) -> /Channels/K19
- Q517 pad 1: /Channels/GA21 -> Net-(Q517-Pad1)
- Q517 pad 2: GND -> 400V
- Q518 pad 1: /Channels/GA22 -> /Channels/GK23
- Q518 pad 3: Net-(Q518-Pad3) -> /Channels/K23
- Q519 pad 1: /Channels/GA23 -> /Channels/GA20
- Q521 pad 1: /Channels/GK21 -> Net-(Q521-Pad1)
- Q521 pad 2: GND -> 400V
- Q521 pad 3: /Channels/K21 -> Net-(Q521-Pad3)
- Q522 pad 1: /Channels/GK22 -> /Channels/GK20
- Q522 pad 3: /Channels/K22 -> /Channels/K20
- Q523 pad 1: /Channels/GK23 -> Net-(Q523-Pad1)
- Q523 pad 2: GND -> 400V
- Q523 pad 3: /Channels/K23 -> Net-(Q523-Pad3)
- Q601 pad 1: Net-(Q601-Pad1) -> /Channels/GA25
- Q601 pad 2: 400V -> GND
- Q602 pad 1: Net-(Q602-Pad1) -> /Channels/GA29
- Q602 pad 2: 400V -> GND
- Q604 pad 1: Net-(Q604-Pad1) -> /Channels/GK25
- Q604 pad 2: 400V -> GND
- Q604 pad 3: Net-(Q604-Pad3) -> /Channels/K25
- Q605 pad 1: /Channels/GA25 -> Net-(Q605-Pad1)
- Q605 pad 2: GND -> 400V
- Q606 pad 1: /Channels/GA26 -> /Channels/GK29
- Q606 pad 3: Net-(Q606-Pad3) -> /Channels/K29
- Q607 pad 1: /Channels/GA27 -> /Channels/GA26
- Q608 pad 1: /Channels/GA28 -> /Channels/GA30
- Q609 pad 1: /Channels/GK25 -> Net-(Q609-Pad1)
- Q609 pad 2: GND -> 400V
- Q609 pad 3: /Channels/K25 -> Net-(Q609-Pad3)
- Q611 pad 1: /Channels/GK27 -> Net-(Q611-Pad1)
- Q611 pad 2: GND -> 400V
- Q611 pad 3: /Channels/K27 -> Net-(Q611-Pad3)
- Q612 pad 1: /Channels/GK28 -> /Channels/GK30
- Q612 pad 3: /Channels/K28 -> /Channels/K30
- Q613 pad 1: Net-(Q613-Pad1) -> /Channels/GA27
- Q613 pad 2: 400V -> GND
- Q614 pad 1: Net-(Q614-Pad1) -> /Channels/GA31
- Q614 pad 2: 400V -> GND
- Q616 pad 1: Net-(Q616-Pad1) -> /Channels/GK27
- Q616 pad 2: 400V -> GND
- Q616 pad 3: Net-(Q616-Pad3) -> /Channels/K27
- Q617 pad 1: /Channels/GA29 -> Net-(Q617-Pad1)
- Q617 pad 2: GND -> 400V
- Q618 pad 1: /Channels/GA30 -> /Channels/GK31
- Q618 pad 3: Net-(Q618-Pad3) -> /Channels/K31
- Q619 pad 1: /Channels/GA31 -> /Channels/GA28
- Q621 pad 1: /Channels/GK29 -> Net-(Q621-Pad1)
- Q621 pad 2: GND -> 400V
- Q621 pad 3: /Channels/K29 -> Net-(Q621-Pad3)
- Q622 pad 1: /Channels/GK30 -> /Channels/GK28
- Q622 pad 3: /Channels/K30 -> /Channels/K28
- Q623 pad 1: /Channels/GK31 -> Net-(Q623-Pad1)
- Q623 pad 2: GND -> 400V
- Q623 pad 3: /Channels/K31 -> Net-(Q623-Pad3)
- R301 pad 1: Net-(Q301-Pad1) -> Net-(Q303-Pad1)
- R301 pad 2: 400V -> Net-(Q301-Pad3)
- R302 pad 1: Net-(Q302-Pad1) -> Net-(Q305-Pad1)
- R302 pad 2: 400V -> Net-(Q302-Pad3)
- R304 pad 1: Net-(Q304-Pad1) -> Net-(Q305-Pad1)
- R305 pad 1: Net-(Q301-Pad1) -> Net-(Q303-Pad3)
- R305 pad 2: Net-(Q305-Pad3) -> /Channels/A1
- R306 pad 1: Net-(Q302-Pad1) -> Net-(Q305-Pad3)
- R306 pad 2: Net-(Q306-Pad3) -> /Channels/A5
- R307 pad 1: Net-(Q303-Pad1) -> Net-(Q309-Pad1)
- R308 pad 1: Net-(Q304-Pad1) -> Net-(Q311-Pad1)
- R309 pad 1: Net-(Q301-Pad3) -> Net-(Q309-Pad1)
- R309 pad 2: /Channels/A1 -> 400V
- R310 pad 1: Net-(Q302-Pad3) -> Net-(Q311-Pad1)
- R310 pad 2: /Channels/A2 -> 400V
- R311 pad 1: Net-(Q303-Pad3) -> Net-(Q309-Pad3)
- R311 pad 2: /Channels/A3 -> /Channels/A2
- R312 pad 1: Net-(Q304-Pad3) -> Net-(Q311-Pad3)
- R312 pad 2: /Channels/A4 -> /Channels/A6
- R313 pad 1: Net-(Q313-Pad1) -> Net-(Q315-Pad1)
- R313 pad 2: 400V -> Net-(Q313-Pad3)
- R314 pad 1: Net-(Q314-Pad1) -> Net-(Q317-Pad1)
- R314 pad 2: 400V -> Net-(Q314-Pad3)
- R316 pad 1: Net-(Q316-Pad1) -> Net-(Q317-Pad1)
- R317 pad 1: Net-(Q313-Pad1) -> Net-(Q315-Pad3)
- R317 pad 2: Net-(Q317-Pad3) -> /Channels/A3
- R318 pad 1: Net-(Q314-Pad1) -> Net-(Q317-Pad3)
- R318 pad 2: Net-(Q318-Pad3) -> /Channels/A7
- R319 pad 1: Net-(Q315-Pad1) -> Net-(Q321-Pad1)
- R320 pad 1: Net-(Q316-Pad1) -> Net-(Q323-Pad1)
- R321 pad 1: Net-(Q313-Pad3) -> Net-(Q321-Pad1)
- R321 pad 2: /Channels/A5 -> 400V
- R322 pad 1: Net-(Q314-Pad3) -> Net-(Q323-Pad1)
- R322 pad 2: /Channels/A6 -> 400V
- R323 pad 1: Net-(Q315-Pad3) -> Net-(Q321-Pad3)
- R323 pad 2: /Channels/A7 -> /Channels/A4
- R324 pad 1: Net-(Q316-Pad3) -> Net-(Q323-Pad3)
- R401 pad 1: Net-(Q401-Pad1) -> Net-(Q403-Pad1)
- R401 pad 2: 400V -> Net-(Q401-Pad3)
- R402 pad 1: Net-(Q402-Pad1) -> Net-(Q405-Pad1)
- R402 pad 2: 400V -> Net-(Q402-Pad3)
- R404 pad 1: Net-(Q404-Pad1) -> Net-(Q405-Pad1)
- R405 pad 1: Net-(Q401-Pad1) -> Net-(Q403-Pad3)
- R405 pad 2: Net-(Q405-Pad3) -> /Channels/A9
- R406 pad 1: Net-(Q402-Pad1) -> Net-(Q405-Pad3)
- R406 pad 2: Net-(Q406-Pad3) -> /Channels/A13
- R407 pad 1: Net-(Q403-Pad1) -> Net-(Q409-Pad1)
- R408 pad 1: Net-(Q404-Pad1) -> Net-(Q411-Pad1)
- R409 pad 1: Net-(Q401-Pad3) -> Net-(Q409-Pad1)
- R409 pad 2: /Channels/A9 -> 400V
- R410 pad 1: Net-(Q402-Pad3) -> Net-(Q411-Pad1)
- R410 pad 2: /Channels/A10 -> 400V
- R411 pad 1: Net-(Q403-Pad3) -> Net-(Q409-Pad3)
- R411 pad 2: /Channels/A11 -> /Channels/A10
- R412 pad 1: Net-(Q404-Pad3) -> Net-(Q411-Pad3)
- R412 pad 2: /Channels/A12 -> /Channels/A14
- R413 pad 1: Net-(Q413-Pad1) -> Net-(Q415-Pad1)
- R413 pad 2: 400V -> Net-(Q413-Pad3)
- R414 pad 1: Net-(Q414-Pad1) -> Net-(Q417-Pad1)
- R414 pad 2: 400V -> Net-(Q414-Pad3)
- R416 pad 1: Net-(Q416-Pad1) -> Net-(Q417-Pad1)
- R417 pad 1: Net-(Q413-Pad1) -> Net-(Q415-Pad3)
- R417 pad 2: Net-(Q417-Pad3) -> /Channels/A11
- R418 pad 1: Net-(Q414-Pad1) -> Net-(Q417-Pad3)
- R418 pad 2: Net-(Q418-Pad3) -> /Channels/A15
- R419 pad 1: Net-(Q415-Pad1) -> Net-(Q421-Pad1)
- R420 pad 1: Net-(Q416-Pad1) -> Net-(Q423-Pad1)
- R421 pad 1: Net-(Q413-Pad3) -> Net-(Q421-Pad1)
- R421 pad 2: /Channels/A13 -> 400V
- R422 pad 1: Net-(Q414-Pad3) -> Net-(Q423-Pad1)
- R422 pad 2: /Channels/A14 -> 400V
- R423 pad 1: Net-(Q415-Pad3) -> Net-(Q421-Pad3)
- R423 pad 2: /Channels/A15 -> /Channels/A12
- R424 pad 1: Net-(Q416-Pad3) -> Net-(Q423-Pad3)
- R501 pad 1: Net-(Q501-Pad1) -> Net-(Q503-Pad1)
- R501 pad 2: 400V -> Net-(Q501-Pad3)
- R502 pad 1: Net-(Q502-Pad1) -> Net-(Q505-Pad1)
- R502 pad 2: 400V -> Net-(Q502-Pad3)
- R504 pad 1: Net-(Q504-Pad1) -> Net-(Q505-Pad1)
- R505 pad 1: Net-(Q501-Pad1) -> Net-(Q503-Pad3)
- R505 pad 2: Net-(Q505-Pad3) -> /Channels/A17
- R506 pad 1: Net-(Q502-Pad1) -> Net-(Q505-Pad3)
- R506 pad 2: Net-(Q506-Pad3) -> /Channels/A21
- R507 pad 1: Net-(Q503-Pad1) -> Net-(Q509-Pad1)
- R508 pad 1: Net-(Q504-Pad1) -> Net-(Q511-Pad1)
- R509 pad 1: Net-(Q501-Pad3) -> Net-(Q509-Pad1)
- R509 pad 2: /Channels/A17 -> 400V
- R510 pad 1: Net-(Q502-Pad3) -> Net-(Q511-Pad1)
- R510 pad 2: /Channels/A18 -> 400V
- R511 pad 1: Net-(Q503-Pad3) -> Net-(Q509-Pad3)
- R511 pad 2: /Channels/A19 -> /Channels/A18
- R512 pad 1: Net-(Q504-Pad3) -> Net-(Q511-Pad3)
- R512 pad 2: /Channels/A20 -> /Channels/A22
- R513 pad 1: Net-(Q513-Pad1) -> Net-(Q515-Pad1)
- R513 pad 2: 400V -> Net-(Q513-Pad3)
- R514 pad 1: Net-(Q514-Pad1) -> Net-(Q517-Pad1)
- R514 pad 2: 400V -> Net-(Q514-Pad3)
- R516 pad 1: Net-(Q516-Pad1) -> Net-(Q517-Pad1)
- R517 pad 1: Net-(Q513-Pad1) -> Net-(Q515-Pad3)
- R517 pad 2: Net-(Q517-Pad3) -> /Channels/A19
- R518 pad 1: Net-(Q514-Pad1) -> Net-(Q517-Pad3)
- R518 pad 2: Net-(Q518-Pad3) -> /Channels/A23
- R519 pad 1: Net-(Q515-Pad1) -> Net-(Q521-Pad1)
- R520 pad 1: Net-(Q516-Pad1) -> Net-(Q523-Pad1)
- R521 pad 1: Net-(Q513-Pad3) -> Net-(Q521-Pad1)
- R521 pad 2: /Channels/A21 -> 400V
- R522 pad 1: Net-(Q514-Pad3) -> Net-(Q523-Pad1)
- R522 pad 2: /Channels/A22 -> 400V
- R523 pad 1: Net-(Q515-Pad3) -> Net-(Q521-Pad3)
- R523 pad 2: /Channels/A23 -> /Channels/A20
- R524 pad 1: Net-(Q516-Pad3) -> Net-(Q523-Pad3)
- R601 pad 1: Net-(Q601-Pad1) -> Net-(Q603-Pad1)
- R601 pad 2: 400V -> Net-(Q601-Pad3)
- R602 pad 1: Net-(Q602-Pad1) -> Net-(Q605-Pad1)
- R602 pad 2: 400V -> Net-(Q602-Pad3)
- R604 pad 1: Net-(Q604-Pad1) -> Net-(Q605-Pad1)
- R605 pad 1: Net-(Q601-Pad1) -> Net-(Q603-Pad3)
- R605 pad 2: Net-(Q605-Pad3) -> /Channels/A25
- R606 pad 1: Net-(Q602-Pad1) -> Net-(Q605-Pad3)
- R606 pad 2: Net-(Q606-Pad3) -> /Channels/A29
- R607 pad 1: Net-(Q603-Pad1) -> Net-(Q609-Pad1)
- R608 pad 1: Net-(Q604-Pad1) -> Net-(Q611-Pad1)
- R609 pad 1: Net-(Q601-Pad3) -> Net-(Q609-Pad1)
- R609 pad 2: /Channels/A25 -> 400V
- R610 pad 1: Net-(Q602-Pad3) -> Net-(Q611-Pad1)
- R610 pad 2: /Channels/A26 -> 400V
- R611 pad 1: Net-(Q603-Pad3) -> Net-(Q609-Pad3)
- R611 pad 2: /Channels/A27 -> /Channels/A26
- R612 pad 1: Net-(Q604-Pad3) -> Net-(Q611-Pad3)
- R612 pad 2: /Channels/A28 -> /Channels/A30
- R613 pad 1: Net-(Q613-Pad1) -> Net-(Q615-Pad1)
- R613 pad 2: 400V -> Net-(Q613-Pad3)
- R614 pad 1: Net-(Q614-Pad1) -> Net-(Q617-Pad1)
- R614 pad 2: 400V -> Net-(Q614-Pad3)
- R616 pad 1: Net-(Q616-Pad1) -> Net-(Q617-Pad1)
- R617 pad 1: Net-(Q613-Pad1) -> Net-(Q615-Pad3)
- R617 pad 2: Net-(Q617-Pad3) -> /Channels/A27
- R618 pad 1: Net-(Q614-Pad1) -> Net-(Q617-Pad3)
- R618 pad 2: Net-(Q618-Pad3) -> /Channels/A31
- R619 pad 1: Net-(Q615-Pad1) -> Net-(Q621-Pad1)
- R620 pad 1: Net-(Q616-Pad1) -> Net-(Q623-Pad1)
- R621 pad 1: Net-(Q613-Pad3) -> Net-(Q621-Pad1)
- R621 pad 2: /Channels/A29 -> 400V
- R622 pad 1: Net-(Q614-Pad3) -> Net-(Q623-Pad1)
- R622 pad 2: /Channels/A30 -> 400V
- R623 pad 1: Net-(Q615-Pad3) -> Net-(Q621-Pad3)
- R623 pad 2: /Channels/A31 -> /Channels/A28
- R624 pad 1: Net-(Q616-Pad3) -> Net-(Q623-Pad3)
- Y101 pad 3: Net-(IC102-Pad5) -> Net-(IC101-Pad5)
Other:
- board size 162.1 x 162.1 mm -> 162 x 162 mm

Commit message: more layout work
Parts:
- added J108: HV, agg:MOLEX-KK-254P-03, F.Cu at (180.0, 84.0)
- added J109: PSU, agg:MOLEX-KK-254P-04, F.Cu at (180.0, 134.5)
- IC102: value TSR 1-2433 -> TSR 1-2450
- moved IC701 255.9 mm to (118.5, 186.5)
- moved IC703 222.7 mm to (118.5, 154.5)
- moved IC705 179.8 mm to (118.5, 112.5)
- moved R501 179.8 mm to (107.0, 136.0)
- moved Q513 176.7 mm to (111.5, 128.5), turned to 180 degrees
- moved Q503 175.6 mm to (96.0, 136.5), turned to 180 degrees
- moved R507 170.9 mm to (107.0, 132.0)
- moved Q515 168.7 mm to (96.0, 128.5), turned to 180 degrees
- moved Q509 168.2 mm to (96.0, 132.5), turned to 180 degrees
- moved R503 168.2 mm to (102.0, 136.0), turned to 180 degrees
- moved Q511 167.9 mm to (96.0, 116.5), turned to 180 degrees
- moved R519 167.8 mm to (107.0, 124.0)
- moved R515 165.1 mm to (102.0, 128.0), turned to 180 degrees
- moved Q508 164.1 mm to (111.5, 116.5), turned to 180 degrees
- moved Q521 163.8 mm to (96.0, 124.5), turned to 180 degrees
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Connections:
- C111 pad 1: 3v3 -> 5v
- IC102 pad 3: 3v3 -> 5v
- IC701 pad 1: /Channels/GA2 -> /Channels/GA7
- IC701 pad 15: /Channels/GA1 -> /Channels/GA8
- IC701 pad 2: /Channels/GA3 -> /Channels/GA6
- IC701 pad 3: /Channels/GA4 -> /Channels/GA5
- IC701 pad 4: /Channels/GA5 -> /Channels/GA4
- IC701 pad 5: /Channels/GA6 -> /Channels/GA3
- IC701 pad 6: /Channels/GA7 -> /Channels/GA2
- IC701 pad 7: /Channels/GA8 -> /Channels/GA1
- IC703 pad 1: /Channels/GA10 -> /Channels/GA15
- IC703 pad 15: /Channels/GA9 -> /Channels/GA16
- IC703 pad 2: /Channels/GA11 -> /Channels/GA14
- IC703 pad 3: /Channels/GA12 -> /Channels/GA13
- IC703 pad 4: /Channels/GA13 -> /Channels/GA12
- IC703 pad 5: /Channels/GA14 -> /Channels/GA11
- IC703 pad 6: /Channels/GA15 -> /Channels/GA10
- IC703 pad 7: /Channels/GA16 -> /Channels/GA9
- IC705 pad 1: /Channels/GA18 -> /Channels/GA23
- IC705 pad 15: /Channels/GA17 -> /Channels/GA24
- IC705 pad 2: /Channels/GA19 -> /Channels/GA22
- IC705 pad 3: /Channels/GA20 -> /Channels/GA21
- IC705 pad 4: /Channels/GA21 -> /Channels/GA20
- IC705 pad 5: /Channels/GA22 -> /Channels/GA19
- IC705 pad 6: /Channels/GA23 -> /Channels/GA18
- IC705 pad 7: /Channels/GA24 -> /Channels/GA17
- IC707 pad 1: /Channels/GA26 -> /Channels/GA31
- IC707 pad 15: /Channels/GA25 -> /Channels/GA32
- IC707 pad 2: /Channels/GA27 -> /Channels/GA30
- IC707 pad 3: /Channels/GA28 -> /Channels/GA29
- IC707 pad 4: /Channels/GA29 -> /Channels/GA28
- IC707 pad 5: /Channels/GA30 -> /Channels/GA27
- IC707 pad 6: /Channels/GA31 -> /Channels/GA26
- IC707 pad 7: /Channels/GA32 -> /Channels/GA25
- J202 pad 10: /Channels/K22 -> /Channels/K24
- J202 pad 12: /Channels/K26 -> /Channels/K22
- J202 pad 6: /Channels/K24 -> /Channels/K28
- J202 pad 8: /Channels/K28 -> /Channels/K26
- TP101 pad 1: 3v3 -> 5v

Commit message: WIP routing driver
Parts:
- added J203: K_1_16, agg:IPL1-116-02-L-SH, F.Cu at (153.5, 52.8)
- added J204: K_1_16, agg:IPL1-116-02-L-SH, F.Cu at (97.5, 52.8)
- J201: value A_1_32 -> A_1_16; footprint agg:DIL-254P-32 -> agg:IPL1-116-02-L-SH
- J202: value K_1_32 -> A_17_32; footprint agg:DIL-254P-32 -> agg:IPL1-116-02-L-SH
- moved C101 256.8 mm to (320.6, 112.5)
- moved C102 256.8 mm to (311.4, 124.1)
- moved C103 256.8 mm to (323.4, 108.4)
- moved C104 256.8 mm to (316.5, 116.3)
- moved C105 256.8 mm to (301.0, 131.9)
- moved C106 256.8 mm to (311.4, 121.6)
- moved C107 256.8 mm to (301.0, 129.4)
- moved C108 256.8 mm to (319.3, 110.0)
- moved C109 256.8 mm to (307.3, 121.6)
- moved C110 256.8 mm to (282.4, 130.7)
- moved C111 256.8 mm to (282.4, 134.9)
- moved C112 256.8 mm to (296.9, 129.4)
- moved C113 256.8 mm to (296.9, 131.9)
- moved C114 256.8 mm to (323.4, 105.9)
- moved C115 256.8 mm to (307.3, 124.1)
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Connections:
- J202 pad 1: /Channels/K31 -> /Channels/A17
- J202 pad 10: /Channels/K24 -> /Channels/A26
- J202 pad 11: /Channels/K21 -> /Channels/A27
- J202 pad 12: /Channels/K22 -> /Channels/A28
- J202 pad 13: /Channels/K19 -> /Channels/A29
- J202 pad 14: /Channels/K20 -> /Channels/A30
- J202 pad 15: /Channels/K17 -> /Channels/A31
- J202 pad 16: /Channels/K18 -> /Channels/A32
- J202 pad 2: /Channels/K32 -> /Channels/A18
- J202 pad 3: /Channels/K29 -> /Channels/A19
- J202 pad 4: /Channels/K30 -> /Channels/A20
- J202 pad 5: /Channels/K27 -> /Channels/A21
- J202 pad 6: /Channels/K28 -> /Channels/A22
- J202 pad 7: /Channels/K25 -> /Channels/A23
- J202 pad 8: /Channels/K26 -> /Channels/A24
- J202 pad 9: /Channels/K23 -> /Channels/A25
Routing:
- net 400V: track 0.00 -> 237.2 mm
- net GND: track 0.00 -> 30.4 mm, vias 0 -> 32
- net /Channels/GK32: track 0.00 -> 27.0 mm
- net /Channels/GK24: track 0.00 -> 26.2 mm
- net /Channels/A8: track 0.00 -> 25.1 mm, vias 0 -> 2
- net /Channels/A32: track 0.00 -> 25.0 mm
- net /Channels/A7: track 0.00 -> 24.0 mm, vias 0 -> 2
- net /Channels/GK31: track 0.00 -> 22.9 mm
- net /Channels/GK23: track 0.00 -> 22.6 mm
- net /Channels/GK30: track 0.00 -> 18.7 mm
- net /Channels/GK22: track 0.00 -> 18.6 mm
- net /Channels/A17: track 0.00 -> 17.9 mm
- net /Channels/A16: track 0.00 -> 17.9 mm
- net /Channels/A1: track 0.00 -> 17.9 mm
- net /Channels/A2: track 0.00 -> 17.3 mm
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